File: Hardware/StepperDriver/Driver/Driver.sch (KiCad schematic (older format))
At the start: 33 parts, among them M1A1 CONN_01X02, M1A2 CONN_01X02, P1 CONN_01X07, Q1 FQP20N06, Q10 2N3704, Q11 FQP20N06, Q12 FQP20N06, Q2 FQP20N06, Q3 2N3704, Q4 2N3704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

Commit message: various production tweaks: fixed track layers and footprints
Parts:
- added H1, H2, H3, H4: CONN_01X01, Mounting_Holes:MountingHole_4mm, symbol CONN_01X01
- D1, D2, D3, D4, D5, D6, D7, D8: footprint Diodes_ThroughHole:Diode_DO-35_SOD27_Horizontal_RM10 -> Diodes_ThroughHole:Diode_DO-201AD_Horizontal_RM15
- Q10, Q3, Q4, Q9: footprint Transistors_OldSowjetAera:OldSowjetaera_Transistor_Type-I_BigPads -> TO_SOT_Packages_THT:TO-92_Molded_Wide
Changed lines of the file:
@@
 F 0 "Q3" H 4460 2320 50  0000 R CNN
 F 1 "2N3704" H 4660 2020 50  0000 R CNN
-F 2 "Transistors_OldSowjetAera:OldSowjetaera_Transistor_Type-I_BigPads" H 4760 2270 29  0001 C CNN
+F 2 "TO_SOT_Packages_THT:TO-92_Molded_Wide" H 4760 2270 29  0001 C CNN
 F 3 "" H 4560 2170 60  0000 C CNN
 	1    4560 2170
@@
 F 0 "Q4" H 6710 2070 50  0000 R CNN
 F 1 "2N3704" H 6760 2320 50  0000 R CNN
-F 2 "Transistors_OldSowjetAera:OldSowjetaera_Transistor_Type-I_BigPads" H 6960 2270 29  0001 C CNN
+F 2 "TO_SOT_Packages_THT:TO-92_Molded_Wide" H 6960 2270 29  0001 C CNN
 F 3 "" H 6760 2170 60  0000 C CNN
 	1    6760 2170
@@
 F 0 "D2" H 6060 2070 50  0000 C CNN
 F 1 "SA5.0A" H 6060 1870 50  0000 C CNN
-F 2 "Diodes_ThroughHole:Diode_DO-35_SOD27_Horizontal_RM10" H 6060 1970 60  0001 C CNN
+F 2 "Diodes_ThroughHole:Diode_DO-201AD_Horizontal_RM15" H 6060 1970 60  0001 C CNN
 F 3 "" H 6060 1970 60  0000 C CNN
 	1    6060 1970
@@
 F 0 "D1" H 5310 2070 50  0000 C CNN
 F 1 "SA5.0A" H 5260 2120 50  0000 C CNN
-F 2 "Diodes_ThroughHole:Diode_DO-35_SOD27_Horizontal_RM10" H 5310 1970 60  0001 C CNN
+F 2 "Diodes_ThroughHole:Diode_DO-201AD_Horizontal_RM15" H 5310 1970 60  0001 C CNN
 F 3 "" H 5310 1970 60  0000 C CNN
 	1    5310 1970
@@
 F 0 "D3" H 5360 2770 50  0000 C CNN
 F 1 "SA5.0A" H 5460 2820 50  0000 C CNN
-F 2 "Diodes_ThroughHole:Diode_DO-35_SOD27_Horizontal_RM10" H 5310 2670 60  0001 C CNN
+F 2 "Diodes_ThroughHole:Diode_DO-201AD_Horizontal_RM15" H 5310 2670 60  0001 C CNN
 F 3 "" H 5310 2670 60  0000 C CNN
 	1    5310 2670
@@
 F 0 "D4" H 6060 2820 50  0000 C CNN
 F 1 "SA5.0A" H 6060 2620 50  0000 C CNN
-F 2 "Diodes_ThroughHole:Diode_DO-35_SOD27_Horizontal_RM10" H 6060 2720 60  0001 C CNN
+F 2 "Diodes_ThroughHole:Diode_DO-201AD_Horizontal_RM15" H 6060 2720 60  0001 C CNN
 F 3 "" H 6060 2720 60  0000 C CNN
 	1    6060 2720
@@
 F 0 "Q9" H 4510 4620 50  0000 R CNN
 F 1 "2N3704" H 4710 4320 50  0000 R CNN
-F 2 "Transistors_OldSowjetAera:OldSowjetaera_Transistor_Type-I_BigPads" H 4810 4570 29  0001 C CNN
+F 2 "TO_SOT_Packages_THT:TO-92_Molded_Wide" H 4810 4570 29  0001 C CNN
 F 3 "" H 4610 4470 60  0000 C CNN
 	1    4610 4470
@@
 F 0 "Q10" H 6760 4370 50  0000 R CNN
 F 1 "2N3704" H 6810 4620 50  0000 R CNN
-F 2 "Transistors_OldSowjetAera:OldSowjetaera_Transistor_Type-I_BigPads" H 7010 4570 29  0001 C CNN
+F 2 "TO_SOT_Packages_THT:TO-92_Molded_Wide" H 7010 4570 29  0001 C CNN
 F 3 "" H 6810 4470 60  0000 C CNN
 	1    6810 4470
@@
 F 0 "D6" H 6110 4370 50  0000 C CNN
 F 1 "SA5.0A" H 6110 4170 50  0000 C CNN
-F 2 "Diodes_ThroughHole:Diode_DO-35_SOD27_Horizontal_RM10" H 6110 4270 60  0001 C CNN
+F 2 "Diodes_ThroughHole:Diode_DO-201AD_Horizontal_RM15" H 6110 4270 60  0001 C CNN
 F 3 "" H 6110 4270 60  0000 C CNN
 	1    6110 4270
@@
 F 0 "D5" H 5360 4370 50  0000 C CNN
 F 1 "SA5.0A" H 5360 4420 50  0000 C CNN
-F 2 "Diodes_ThroughHole:Diode_DO-35_SOD27_Horizontal_RM10" H 5360 4270 60  0001 C CNN
+F 2 "Diodes_ThroughHole:Diode_DO-201AD_Horizontal_RM15" H 5360 4270 60  0001 C CNN
 F 3 "" H 5360 4270 60  0000 C CNN
 	1    5360 4270
@@
 F 0 "D7" H 5410 5070 50  0000 C CNN
 F 1 "SA5.0A" H 5460 5120 50  0000 C CNN
-F 2 "Diodes_ThroughHole:Diode_DO-35_SOD27_Horizontal_RM10" H 5360 4970 60  0001 C CNN
+F 2 "Diodes_ThroughHole:Diode_DO-201AD_Horizontal_RM15" H 5360 4970 60  0001 C CNN
 F 3 "" H 5360 4970 60  0000 C CNN
 	1    5360 4970
@@
 F 0 "D8" H 6110 5120 50  0000 C CNN
 F 1 "SA5.0A" H 6110 4920 50  0000 C CNN
-F 2 "Diodes_ThroughHole:Diode_DO-35_SOD27_Horizontal_RM10" H 6110 5020 60  0001 C CNN
+F 2 "Diodes_ThroughHole:Diode_DO-201AD_Horizontal_RM15" H 6110 5020 60  0001 C CNN
 F 3 "" H 6110 5020 60  0000 C CNN
 	1    6110 5020
@@
 Text Label 3910 5020 2    60   ~ 0
 STEPPER1PHASEB1
+$Comp
+L CONN_01X01 H1
+U 1 1 56A63CAE
+P 1880 6530
+F 0 "H1" H 1880 6630 50  0000 C CNN
+F 1 "CONN_01X01" V 1980 6530 50  0000 C CNN
+F 2 "Mounting_Holes:MountingHole_4mm" H 1880 6530 50  0001 C CNN
+F 3 "" H 1880 6530 50  0000 C CNN
+	1    1880 6530
+	1    0    0    -1
+$EndComp
+$Comp
+L CONN_01X01 H4
+U 1 1 56A64097
+P 1870 7040
+F 0 "H4" H 1870 7140 50  0000 C CNN
+F 1 "CONN_01X01" V 1970 7040 50  0000 C CNN
+F 2 "Mounting_Holes:MountingHole_4mm" H 1870 7040 50  0001 C CNN
+F 3 "" H 1870 7040 50  0000 C CNN
+	1    1870 7040
+	1    0    0    -1
+$EndComp
+$Comp
+L CONN_01X01 H2
+U 1 1 56A6414E
+P 2430 6530
+F 0 "H2" H 2430 6630 50  0000 C CNN
+F 1 "CONN_01X01" V 2530 6530 50  0000 C CNN
+F 2 "Mounting_Holes:MountingHole_4mm" H 2430 6530 50  0001 C CNN
+F 3 "" H 2430 6530 50  0000 C CNN
+	1    2430 6530
+	1    0    0    -1
+$EndComp
+$Comp
+L CONN_01X01 H3
+U 1 1 56A6422E
+P 2430 7070
+F 0 "H3" H 2430 7170 50  0000 C CNN
+F 1 "CONN_01X01" V 2530 7070 50  0000 C CNN
+F 2 "Mounting_Holes:MountingHole_4mm" H 2430 7070 50  0001 C CNN
+F 3 "" H 2430 7070 50  0000 C CNN
+	1    2430 7070
+	1    0    0    -1
+$EndComp
 $EndSCHEMATC
