File: Hardware/StepperDriver/Driver/Driver.kicad_pcb (KiCad board)
At the start: 2 copper layers, 97.6 x 107.1 mm, 37 parts, among them M1A1 CONN_01X02, M1A2 CONN_01X02, P1 CONN_01X07, Q1 FQP20N06, Q10 2N3704, Q11 FQP20N06, Q12 FQP20N06, Q2 FQP20N06, Q3 2N3704, Q4 2N3704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

Commit message: added quick and dirty keepout zones to the solder Resist layer added board identification text added alignment marks to other layers (solder resist + Silk)
Other:
- board text added: "Stepper Driver Rev. A 2016 Flow Project"
