File: Hardware/StepperDriver/Brains/Brains.sch (KiCad schematic (older format))
At the start: 14 parts, among them IC1 ATMEGA328-P, P1 CONN_01X02, P2 CONN_01X02, P3 CONN_01X07, P4 CONN_01X07, P5 CONN_01X07, P6 CONN_01X04, Y1 Crystal

Commit message: fixed incorrect Xtal footprint
Parts:
- Y1: footprint Crystals:Crystal_HC48-U_Vertical -> Crystals:Crystal_HC49-U_Vertical
Changed lines of the file:
@@
 F 0 "Y1" H 7210 4000 50  0000 C CNN
 F 1 "Crystal" H 7210 3700 50  0000 C CNN
-F 2 "Crystals:Crystal_HC48-U_Vertical" H 7210 3850 60  0001 C CNN
+F 2 "Crystals:Crystal_HC49-U_Vertical" H 7210 3850 60  0001 C CNN
 F 3 "" H 7210 3850 60  0000 C CNN
 	1    7210 3850
