File: Hardware/HotWireADC/Rev2/HotWireRev2.sch (KiCad schematic (older format))
At the start: 48 parts, among them CON1 BARREL_JACK, P1 BNC, P2 BNC, P3 BNC, P4 BNC, P5 CONN_02X06, P6 BNC, SW1 SW_PUSH_SMALL, U1 OPA320, U2 OPA320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

Commit message: updated component names and created BOM
Parts:
- C9: value 10u -> 10u tant
- R10: value 0.5 -> 0.5R
Changed lines of the file:
@@
 P 8920 3160
 F 0 "R10" H 8950 3180 50  0000 L CNN
-F 1 "0.5" H 8950 3120 50  0000 L CNN
+F 1 "0.5R" H 8950 3120 50  0000 L CNN
 F 2 "Resistors_SMD:R_1206_HandSoldering" H 8920 3160 50  0001 C CNN
 F 3 "" H 8920 3160 50  0000 C CNN
@@
 P 6720 4860
 F 0 "C9" H 6730 4930 50  0000 L CNN
-F 1 "10u" H 6730 4780 50  0000 L CNN
+F 1 "10u tant" H 6730 4780 50  0000 L CNN
 F 2 "Capacitors_Tantalum_SMD:TantalC_SizeU_EIA-6032" H 6720 4860 50  0001 C CNN
 F 3 "" H 6720 4860 50  0000 C CNN
@@
 IN1
 $Comp
-L GNDA #PWR024
+L GNDA #PWR023
 U 1 1 56E89E10
 P 1400 6040
-F 0 "#PWR024" H 1400 5790 50  0001 C CNN
+F 0 "#PWR023" H 1400 5790 50  0001 C CNN
 F 1 "GNDA" H 1400 5890 50  0000 C CNN
 F 2 "" H 1400 6040 50  0000 C CNN
@@
 Connection ~ 3240 6280
 $Comp
-L GNDA #PWR025
+L GNDA #PWR024
 U 1 1 56E8E642
 P 1720 7310
-F 0 "#PWR025" H 1720 7060 50  0001 C CNN
+F 0 "#PWR024" H 1720 7060 50  0001 C CNN
 F 1 "GNDA" H 1720 7160 50  0000 C CNN
 F 2 "" H 1720 7310 50  0000 C CNN
@@
 $EndComp
 $Comp
-L +3.3V #PWR026
+L +3.3V #PWR025
 U 1 1 56E902E0
 P 3800 6190
-F 0 "#PWR026" H 3800 6040 50  0001 C CNN
+F 0 "#PWR025" H 3800 6040 50  0001 C CNN
 F 1 "+3.3V" H 3800 6330 50  0000 C CNN
 F 2 "" H 3800 6190 50  0000 C CNN
@@
 $EndComp
 $Comp
-L GNDA #PWR027
+L GNDA #PWR026
 U 1 1 56E93599
 P 8960 5880
-F 0 "#PWR027" H 8960 5630 50  0001 C CNN
+F 0 "#PWR026" H 8960 5630 50  0001 C CNN
 F 1 "GNDA" H 8960 5730 50  0000 C CNN
 F 2 "" H 8960 5880 50  0000 C CNN
@@
 Connection ~ 8960 5800
 $Comp
-L VCC #PWR028
+L VCC #PWR027
 U 1 1 56E941B0
 P 8970 5530
-F 0 "#PWR028" H 8970 5380 50  0001 C CNN
+F 0 "#PWR027" H 8970 5380 50  0001 C CNN
 F 1 "VCC" H 8970 5680 50  0000 C CNN
 F 2 "" H 8970 5530 50  0000 C CNN
@@
 	8970 5600 8970 5530
 $Comp
-L PWR_FLAG #FLG029
+L PWR_FLAG #FLG028
 U 1 1 56E94ED5
 P 8810 5450
-F 0 "#FLG029" H 8810 5545 50  0001 C CNN
+F 0 "#FLG028" H 8810 5545 50  0001 C CNN
 F 1 "PWR_FLAG" H 8810 5630 50  0000 C CNN
 F 2 "" H 8810 5450 50  0000 C CNN
@@
 $EndComp
 $Comp
-L PWR_FLAG #FLG030
+L PWR_FLAG #FLG029
 U 1 1 56E95487
 P 9220 5700
-F 0 "#FLG030" H 9220 5795 50  0001 C CNN
+F 0 "#FLG029" H 9220 5795 50  0001 C CNN
 F 1 "PWR_FLAG" H 9220 5880 50  0000 C CNN
 F 2 "" H 9220 5700 50  0000 C CNN
@@
 $EndComp
 $Comp
-L PWR_FLAG #FLG031
+L PWR_FLAG #FLG030
 U 1 1 56E957F2
 P 4110 6240
-F 0 "#FLG031" H 4110 6335 50  0001 C CNN
+F 0 "#FLG030" H 4110 6335 50  0001 C CNN
 F 1 "PWR_FLAG" H 4110 6420 50  0000 C CNN
 F 2 "" H 4110 6240 50  0000 C CNN
@@
 Connection ~ 8890 5600
 $Comp
-L GNDD #PWR032
+L GNDD #PWR031
 U 1 1 56E9B38E
 P 3150 6620
-F 0 "#PWR032" H 3150 6370 50  0001 C CNN
+F 0 "#PWR031" H 3150 6370 50  0001 C CNN
 F 1 "GNDD" H 3150 6470 50  0000 C CNN
 F 2 "" H 3150 6620 50  0000 C CNN
@@
 Connection ~ 3150 6540
 $Comp
-L GNDD #PWR033
+L GNDD #PWR032
 U 1 1 56E9D5EC
 P 2080 7320
-F 0 "#PWR033" H 2080 7070 50  0001 C CNN
+F 0 "#PWR032" H 2080 7070 50  0001 C CNN
 F 1 "GNDD" H 2080 7170 50  0000 C CNN
 F 2 "" H 2080 7320 50  0000 C CNN
@@
 EXT_REF
 $Comp
-L GNDA #PWR034
+L GNDA #PWR033
 U 1 1 56EAC6C3
 P 8410 3420
-F 0 "#PWR034" H 8410 3170 50  0001 C CNN
+F 0 "#PWR033" H 8410 3170 50  0001 C CNN
 F 1 "GNDA" H 8410 3270 50  0000 C CNN
 F 2 "" H 8410 3420 50  0000 C CNN
@@
 	8410 3330 8410 3420
 $Comp
-L +5VA #PWR035
+L +5VA #PWR034
 U 1 1 56EAD0BF
 P 8410 2510
-F 0 "#PWR035" H 8410 2360 50  0001 C CNN
+F 0 "#PWR034" H 8410 2360 50  0001 C CNN
 F 1 "+5VA" H 8410 2650 50  0000 C CNN
 F 2 "" H 8410 2510 50  0000 C CNN
@@
 $EndComp
 $Comp
-L GNDA #PWR036
+L GNDA #PWR035
 U 1 1 56E5C590
 P 4950 6120
-F 0 "#PWR036" H 4950 5870 50  0001 C CNN
+F 0 "#PWR035" H 4950 5870 50  0001 C CNN
 F 1 "GNDA" H 4950 5970 50  0000 C CNN
 F 2 "" H 4950 6120 50  0000 C CNN

Commit message: updated schematic to use correct DC jack footprint
Parts:
- CON1: footprint Connect:JACK_ALIM -> CustomFootprints:JACK_SMD
Changed lines of the file:
@@
 F 0 "CON1" H 8510 5950 50  0000 C CNN
 F 1 "BARREL_JACK" H 8510 5500 50  0000 C CNN
-F 2 "Connect:JACK_ALIM" H 8510 5700 50  0001 C CNN
+F 2 "CustomFootprints:JACK_SMD" H 8510 5700 50  0001 C CNN
 F 3 "" H 8510 5700 50  0000 C CNN
 	1    8510 5700
